File: ESP86266_Bathroom_Edition.kicad_pcb (KiCad board)
At the start: 2 copper layers, 34.9 x 54.6 mm, 17 parts, among them P1 CONN_01X02, P2 CONN_01X04, P3 CONN_01X08, P4 CONN_01X08, P5 CONN_01X04, U1 LM317AH, U2 ESP86266, U3 MCP23017

Commit message: Second version, added M3 mounting holes
Parts:
- added REF**: 1pin, Connect:1pin, F.Cu at (100.3, 121.3)
- added REF**: 1pin, Connect:1pin, F.Cu at (130.2, 121.3)
- added REF**: 1pin, Connect:1pin, F.Cu at (130.2, 71.8)
- added REF**: 1pin, Connect:1pin, F.Cu at (100.3, 71.8)
Changed lines of the file:
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@@
 (kicad_pcb (version 4) (host pcbnew 4.0.0-rc1-stable)
   (general
-    (links 53)
-    (no_connects 1)
+    (links 0)
+    (no_connects 0)
     (area 95.021667 60.729999 135.815 131.090001)
     (thickness 1.6)
@@
     (tracks 248)
     (zones 0)
-    (modules 17)
+    (modules 21)
     (nets 31)
   )
@@
     (pad_to_mask_clearance 0.2)
     (aux_axis_origin 0 0)
-    (visible_elements FFFFFF7F)
+    (visible_elements 7FFFFFFF)
     (pcbplotparams
       (layerselection 0x00030_80000001)
@@
     (add_net "Net-(U3-Pad20)")
   )
+  (module Connect:1pin (layer F.Cu)
+    (at 100.33 121.285)
+    (descr "module 1 pin (ou trou mecanique de percage)")
+    (tags DEV)
+    (fp_text reference REF** (at 0 -3.048) (layer F.SilkS)
+      (effects (font (size 1 1) (thickness 0.15)))
+    )
+    (fp_text value 1pin (at 0 2.794) (layer F.Fab)
+      (effects (font (size 1 1) (thickness 0.15)))
+    )
+    (fp_circle (center 0 0) (end 0 -2.286) (layer F.SilkS) (width 0.15))
+    (pad 1 thru_hole circle (at 0 0) (size 4.064 4.064) (drill 3.048) (layers *.Cu *.Mask F.SilkS))
+  )
+  (module Connect:1pin (layer F.Cu)
+    (at 130.175 121.285)
+    (descr "module 1 pin (ou trou mecanique de percage)")
+    (tags DEV)
+    (fp_text reference REF** (at 0 -3.048) (layer F.SilkS)
+      (effects (font (size 1 1) (thickness 0.15)))
+    )
+    (fp_text value 1pin (at 0 2.794) (layer F.Fab)
+      (effects (font (size 1 1) (thickness 0.15)))
+    )
+    (fp_circle (center 0 0) (end 0 -2.286) (layer F.SilkS) (width 0.15))
+    (pad 1 thru_hole circle (at 0 0) (size 4.064 4.064) (drill 3.048) (layers *.Cu *.Mask F.SilkS))
+  )
+  (module Connect:1pin (layer F.Cu)
+    (at 130.175 71.755)
+    (descr "module 1 pin (ou trou mecanique de percage)")
+    (tags DEV)
+    (fp_text reference REF** (at 0 -3.048) (layer F.SilkS)
+      (effects (font (size 1 1) (thickness 0.15)))
+    )
+    (fp_text value 1pin (at 0 2.794) (layer F.Fab)
+      (effects (font (size 1 1) (thickness 0.15)))
+    )
+    (fp_circle (center 0 0) (end 0 -2.286) (layer F.SilkS) (width 0.15))
+    (pad 1 thru_hole circle (at 0 0) (size 4.064 4.064) (drill 3.048) (layers *.Cu *.Mask F.SilkS))
+  )
   (module Capacitors_SMD:c_elec_8x10 (layer F.Cu)
     (at 119.38 83.1088 90)
@@
     )
   )
+  (module Connect:1pin (layer F.Cu)
+    (at 100.33 71.755)
+    (descr "module 1 pin (ou trou mecanique de percage)")
+    (tags DEV)
+    (fp_text reference REF** (at 0 -3.048) (layer F.SilkS)
+      (effects (font (size 1 1) (thickness 0.15)))
+    )
+    (fp_text value 1pin (at 0 2.794) (layer F.Fab)
+      (effects (font (size 1 1) (thickness 0.15)))
+    )
+    (fp_circle (center 0 0) (end 0 -2.286) (layer F.SilkS) (width 0.15))
+    (pad 1 thru_hole circle (at 0 0) (size 4.064 4.064) (drill 3.048) (layers *.Cu *.Mask F.SilkS))
+  )
   (gr_line (start 97.79 69.215) (end 97.79 123.825) (layer Edge.Cuts) (width 0.15))
